Commit message: modify urdf, visualizer working correctly

File: examples/quad_tilt_wing/quad_tilt_wing.urdf (robot description, URDF)
Before this commit: robot quad_tilt_wing, 17 links, 16 joints
Links:
- link fuselage: mass None -> 0.1
- link wing_1_motor: mass None -> 0.1
- link wing_1_prop: mass None -> 0.1
- link wing_1_rod: mass None -> 0.1
- link wing_1_wing: mass None -> 0.1
- link wing_2_motor: mass None -> 0.1
- link wing_2_prop: mass None -> 0.1
- link wing_2_rod: mass None -> 0.1
- link wing_2_wing: mass None -> 0.1
- link wing_3_motor: mass None -> 0.1
- link wing_3_prop: mass None -> 0.1
- link wing_3_rod: mass None -> 0.1
- link wing_3_wing: mass None -> 0.1
- link wing_4_motor: mass None -> 0.1
- link wing_4_prop: mass None -> 0.1
- link wing_4_rod: mass None -> 0.1
- link wing_4_wing: mass None -> 0.1

File: examples/quad_tilt_wing/quad_tilt_wing.urdf.xacro (robot description, xacro)
@@ -32,4 +32,9 @@
   </material>
   <link name="fuselage">
+    <inertial>
+      <mass value="0.1"/>
+      <origin xyz="0 0 0"/>
+      <inertia ixx="0.01" ixy="0.0" ixz="0.0" iyy="0.01" iyz="0.0" izz="0.01"/>
+    </inertial>
     <visual>
       <geometry>
@@ -40,4 +45,9 @@
   </link>
   <link name="wing_1_rod">
+    <inertial>
+      <mass value="0.1"/>
+      <origin xyz="0 0 0"/>
+      <inertia ixx="0.01" ixy="0.0" ixz="0.0" iyy="0.01" iyz="0.0" izz="0.01"/>
+    </inertial>
     <visual>
       <geometry>
@@ -56,4 +66,9 @@
   </joint>
   <link name="wing_1_wing">
+    <inertial>
+      <mass value="0.1"/>
+      <origin xyz="0 0 0"/>
+      <inertia ixx="0.01" ixy="0.0" ixz="0.0" iyy="0.01" iyz="0.0" izz="0.01"/>
+    </inertial>
     <visual>
       <geometry>
@@ -70,4 +85,9 @@
   </joint>
   <link name="wing_1_motor">
+    <inertial>
+      <mass value="0.1"/>
+      <origin xyz="0 0 0"/>
+      <inertia ixx="0.01" ixy="0.0" ixz="0.0" iyy="0.01" iyz="0.0" izz="0.01"/>
+    </inertial>
     <visual>
       <geometry>
@@ -84,4 +104,9 @@
   </joint>
   <link name="wing_1_prop">
+    <inertial>
+      <mass value="0.1"/>
+      <origin xyz="0 0 0"/>
+      <inertia ixx="0.01" ixy="0.0" ixz="0.0" iyy="0.01" iyz="0.0" izz="0.01"/>
+    </inertial>
     <visual>
       <geometry>
@@ -98,4 +123,9 @@
   </joint>
   <link name="wing_2_rod">
+    <inertial>
+      <mass value="0.1"/>
+      <origin xyz="0 0 0"/>
+      <inertia ixx="0.01" ixy="0.0" ixz="0.0" iyy="0.01" iyz="0.0" izz="0.01"/>
+    </inertial>
     <visual>
       <geometry>
@@ -114,4 +144,9 @@
   </joint>
   <link name="wing_2_wing">
+    <inertial>
+      <mass value="0.1"/>
+      <origin xyz="0 0 0"/>
+      <inertia ixx="0.01" ixy="0.0" ixz="0.0" iyy="0.01" iyz="0.0" izz="0.01"/>
+    </inertial>
     <visual>
       <geometry>
@@ -128,4 +163,9 @@
   </joint>
   <link name="wing_2_motor">
+    <inertial>
+      <mass value="0.1"/>
+      <origin xyz="0 0 0"/>
+      <inertia ixx="0.01" ixy="0.0" ixz="0.0" iyy="0.01" iyz="0.0" izz="0.01"/>
+    </inertial>
     <visual>
       <geometry>
@@ -142,4 +182,9 @@
   </joint>
   <link name="wing_2_prop">
+    <inertial>
+      <mass value="0.1"/>
+      <origin xyz="0 0 0"/>
+      <inertia ixx="0.01" ixy="0.0" ixz="0.0" iyy="0.01" iyz="0.0" izz="0.01"/>
+    </inertial>
     <visual>
       <geometry>
@@ -156,4 +201,9 @@
   </joint>
   <link name="wing_3_rod">
+    <inertial>
+      <mass value="0.1"/>
+      <origin xyz="0 0 0"/>
+      <inertia ixx="0.01" ixy="0.0" ixz="0.0" iyy="0.01" iyz="0.0" izz="0.01"/>
+    </inertial>
     <visual>
       <geometry>
@@ -172,4 +222,9 @@
   </joint>
   <link name="wing_3_wing">
+    <inertial>
+      <mass value="0.1"/>
+      <origin xyz="0 0 0"/>
+      <inertia ixx="0.01" ixy="0.0" ixz="0.0" iyy="0.01" iyz="0.0" izz="0.01"/>
+    </inertial>
     <visual>
       <geometry>
@@ -186,4 +241,9 @@
   </joint>
   <link name="wing_3_motor">
+    <inertial>
+      <mass value="0.1"/>
+      <origin xyz="0 0 0"/>
+      <inertia ixx="0.01" ixy="0.0" ixz="0.0" iyy="0.01" iyz="0.0" izz="0.01"/>
+    </inertial>
     <visual>
       <geometry>
@@ -200,4 +260,9 @@
   </joint>
   <link name="wing_3_prop">
+    <inertial>
+      <mass value="0.1"/>
+      <origin xyz="0 0 0"/>
+      <inertia ixx="0.01" ixy="0.0" ixz="0.0" iyy="0.01" iyz="0.0" izz="0.01"/>
+    </inertial>
     <visual>
       <geometry>
@@ -214,4 +279,9 @@
   </joint>
   <link name="wing_4_rod">
+    <inertial>
+      <mass value="0.1"/>
+      <origin xyz="0 0 0"/>
+      <inertia ixx="0.01" ixy="0.0" ixz="0.0" iyy="0.01" iyz="0.0" izz="0.01"/>
+    </inertial>
     <visual>
       <geometry>
@@ -230,4 +300,9 @@
   </joint>
   <link name="wing_4_wing">
+    <inertial>
+      <mass value="0.1"/>
+      <origin xyz="0 0 0"/>
+      <inertia ixx="0.01" ixy="0.0" ixz="0.0" iyy="0.01" iyz="0.0" izz="0.01"/>
+    </inertial>
     <visual>
       <geometry>
@@ -244,4 +319,9 @@
   </joint>
   <link name="wing_4_motor">
+    <inertial>
+      <mass value="0.1"/>
+      <origin xyz="0 0 0"/>
+      <inertia ixx="0.01" ixy="0.0" ixz="0.0" iyy="0.01" iyz="0.0" izz="0.01"/>
+    </inertial>
     <visual>
       <geometry>
@@ -258,4 +338,9 @@
   </joint>
   <link name="wing_4_prop">
+    <inertial>
+      <mass value="0.1"/>
+      <origin xyz="0 0 0"/>
+      <inertia ixx="0.01" ixy="0.0" ixz="0.0" iyy="0.01" iyz="0.0" izz="0.01"/>
+    </inertial>
     <visual>
       <geometry>

Commit message: modify dynamics, modify urdf file, modify coordinate systems

File: examples/quad_tilt_wing/quad_tilt_wing.urdf (robot description, URDF)
Before this commit: robot quad_tilt_wing, 17 links, 16 joints
Links:
- added link top_indicator, mass 0.1; visual box size=0.5 0.05 0.025
Joints:
- added joint top_to_fuselage: type fixed, parent fuselage, child top_indicator, origin xyz=0.25 0 0.0375
- joint wing_1_joint: axis 0 -1 0 -> 0 1 0; limit lower=-0.523598775598 upper=2.09439510239 effort=1000.0 velocity=0.5 -> lower=-2.09439510239 upper=0.523598775598 effort=1000.0 velocity=0.5
- joint wing_2_joint: axis 0 -1 0 -> 0 1 0; limit lower=-0.523598775598 upper=2.09439510239 effort=1000.0 velocity=0.5 -> lower=-2.09439510239 upper=0.523598775598 effort=1000.0 velocity=0.5
- joint wing_3_joint: axis 0 -1 0 -> 0 1 0; limit lower=-0.523598775598 upper=2.09439510239 effort=1000.0 velocity=0.5 -> lower=-2.09439510239 upper=0.523598775598 effort=1000.0 velocity=0.5
- joint wing_4_joint: axis 0 -1 0 -> 0 1 0; limit lower=-0.523598775598 upper=2.09439510239 effort=1000.0 velocity=0.5 -> lower=-2.09439510239 upper=0.523598775598 effort=1000.0 velocity=0.5

File: examples/quad_tilt_wing/quad_tilt_wing.urdf.xacro (robot description, xacro)
@@ -44,4 +44,22 @@
     </visual>
   </link>
+  <link name="top_indicator">
+    <inertial>
+      <mass value="0.1"/>
+      <origin xyz="0 0 0"/>
+      <inertia ixx="0.01" ixy="0.0" ixz="0.0" iyy="0.01" iyz="0.0" izz="0.01"/>
+    </inertial>
+    <visual>
+      <geometry>
+        <box size="${fuselage_length/2} ${fuselage_height} ${fuselage_height/2}"/>
+      </geometry>
+      <material name="white"/>
+    </visual>
+  </link>
+  <joint name="top_to_fuselage" type="fixed">
+    <parent link="fuselage"/>
+    <child link="top_indicator"/>
+    <origin xyz="${fuselage_length/4} 0 ${fuselage_height/4*3}"/>
+  </joint>
   <link name="wing_1_rod">
     <inertial>
@@ -59,6 +77,6 @@
   </link>
   <joint name="wing_1_joint" type="revolute">
-    <axis xyz="0 -1 0"/>
-    <limit effort="1000.0" lower="-${pi/6}" upper="${2/3*pi}" velocity="0.5"/>
+    <axis xyz="0 1 0"/>
+    <limit effort="1000.0" lower="-${2/3*pi}" upper="${pi/6}" velocity="0.5"/>
     <parent link="fuselage"/>
     <child link="wing_1_rod"/>
@@ -137,6 +155,6 @@
   </link>
   <joint name="wing_2_joint" type="revolute">
-    <axis xyz="0 -1 0"/>
-    <limit effort="1000.0" lower="-${pi/6}" upper="${2/3*pi}" velocity="0.5"/>
+    <axis xyz="0 1 0"/>
+    <limit effort="1000.0" lower="-${2/3*pi}" upper="${pi/6}" velocity="0.5"/>
     <parent link="fuselage"/>
     <child link="wing_2_rod"/>
@@ -215,6 +233,6 @@
   </link>
   <joint name="wing_3_joint" type="revolute">
-    <axis xyz="0 -1 0"/>
-    <limit effort="1000.0" lower="-${pi/6}" upper="${2/3*pi}" velocity="0.5"/>
+    <axis xyz="0 1 0"/>
+    <limit effort="1000.0" lower="-${2/3*pi}" upper="${pi/6}" velocity="0.5"/>
     <parent link="fuselage"/>
     <child link="wing_3_rod"/>
@@ -293,6 +311,6 @@
   </link>
   <joint name="wing_4_joint" type="revolute">
-    <axis xyz="0 -1 0"/>
-    <limit effort="1000.0" lower="-${pi/6}" upper="${2/3*pi}" velocity="0.5"/>
+    <axis xyz="0 1 0"/>
+    <limit effort="1000.0" lower="-${2/3*pi}" upper="${pi/6}" velocity="0.5"/>
     <parent link="fuselage"/>
     <child link="wing_4_rod"/>

Commit message: Add LQR for upright and wing tilt

File: examples/quad_tilt_wing/quad_tilt_wing.urdf (robot description, URDF)
Before this commit: robot quad_tilt_wing, 18 links, 17 joints
Joints:
- joint wing_1_joint: limit lower=-2.09439510239 upper=0.523598775598 effort=1000.0 velocity=0.5 -> lower=-2.35619449019 upper=0.785398163397 effort=1000.0 velocity=0.5
- joint wing_2_joint: limit lower=-2.09439510239 upper=0.523598775598 effort=1000.0 velocity=0.5 -> lower=-2.35619449019 upper=0.785398163397 effort=1000.0 velocity=0.5
- joint wing_3_joint: limit lower=-2.09439510239 upper=0.523598775598 effort=1000.0 velocity=0.5 -> lower=-2.35619449019 upper=0.785398163397 effort=1000.0 velocity=0.5
- joint wing_4_joint: limit lower=-2.09439510239 upper=0.523598775598 effort=1000.0 velocity=0.5 -> lower=-2.35619449019 upper=0.785398163397 effort=1000.0 velocity=0.5

File: examples/quad_tilt_wing/quad_tilt_wing.urdf.xacro (robot description, xacro)
@@ -78,5 +78,5 @@
   <joint name="wing_1_joint" type="revolute">
     <axis xyz="0 1 0"/>
-    <limit effort="1000.0" lower="-${2/3*pi}" upper="${pi/6}" velocity="0.5"/>
+    <limit effort="1000.0" lower="-${pi/2+pi/4}" upper="${pi/4}" velocity="0.5"/>
     <parent link="fuselage"/>
     <child link="wing_1_rod"/>
@@ -156,5 +156,5 @@
   <joint name="wing_2_joint" type="revolute">
     <axis xyz="0 1 0"/>
-    <limit effort="1000.0" lower="-${2/3*pi}" upper="${pi/6}" velocity="0.5"/>
+    <limit effort="1000.0" lower="-${3/4*pi}" upper="${pi/4}" velocity="0.5"/>
     <parent link="fuselage"/>
     <child link="wing_2_rod"/>
@@ -234,5 +234,5 @@
   <joint name="wing_3_joint" type="revolute">
     <axis xyz="0 1 0"/>
-    <limit effort="1000.0" lower="-${2/3*pi}" upper="${pi/6}" velocity="0.5"/>
+    <limit effort="1000.0" lower="-${3/4*pi}" upper="${pi/4}" velocity="0.5"/>
     <parent link="fuselage"/>
     <child link="wing_3_rod"/>
@@ -312,5 +312,5 @@
   <joint name="wing_4_joint" type="revolute">
     <axis xyz="0 1 0"/>
-    <limit effort="1000.0" lower="-${2/3*pi}" upper="${pi/6}" velocity="0.5"/>
+    <limit effort="1000.0" lower="-${3/4*pi}" upper="${pi/4}" velocity="0.5"/>
     <parent link="fuselage"/>
     <child link="wing_4_rod"/>
